Commit message: update code

File: src/my_robot_moveit_config/config/my_robot.ros2_control.xacro (robot description, xacro)
@@ -3,52 +3,59 @@
     <xacro:macro name="my_robot_ros2_control" params="name initial_positions_file">
         <xacro:property name="initial_positions" value="${xacro.load_yaml(initial_positions_file)['initial_positions']}"/>
+        <xacro:arg name="use_mock_component" default="true"/>
         <ros2_control name="${name}" type="system">
             <hardware>
-                <!-- By default, set up controllers for simulation. This won't work on real hardware -->
-                <plugin>mock_components/GenericSystem</plugin>
-            </hardware>
-            <joint name="joint1">
-                <command_interface name="position"/>
-                <state_interface name="position">
-                  <param name="initial_value">${initial_positions['joint1']}</param>
-                </state_interface>
-            </joint>
-            <joint name="joint2">
-                <command_interface name="position"/>
-                <state_interface name="position">
-                  <param name="initial_value">${initial_positions['joint2']}</param>
-                </state_interface>
-            </joint>
-            <joint name="joint3">
-                <command_interface name="position"/>
-                <state_interface name="position">
-                  <param name="initial_value">${initial_positions['joint3']}</param>
-                </state_interface>
-            </joint>
-            <joint name="joint4">
-                <command_interface name="position"/>
-                <state_interface name="position">
-                  <param name="initial_value">${initial_positions['joint4']}</param>
-                </state_interface>
-            </joint>
-            <joint name="joint5">
-                <command_interface name="position"/>
-                <state_interface name="position">
-                  <param name="initial_value">${initial_positions['joint5']}</param>
-                </state_interface>
-            </joint>
-            <joint name="joint6">
-                <command_interface name="position"/>
-                <state_interface name="position">
-                  <param name="initial_value">${initial_positions['joint6']}</param>
-                </state_interface>
-            </joint>
-            <joint name="gripper_left_finger_joint">
-                <command_interface name="position"/>
-                <state_interface name="position">
-                  <param name="initial_value">${initial_positions['gripper_left_finger_joint']}</param>
-                </state_interface>
-            </joint>
-        </ros2_control>
-    </xacro:macro>
-</robot>
+                <xacro:if value="$(arg use_mock_component)">
+                    <plugin>mock_components/GenericSystem</plugin>
+                </xacro:if>
+                <xacro:unless value="$(arg use_mock_component)">
+                    <plugin>arm_hardware/ArmHardwareInterface</plugin>
+                    <param name="joint1_motor_id">10</param>
+                    <param name="joint2_motor_id">20</param>
+                    <param name="dynamixel_port">/dev/ttyACM0</param>
+                </xacro:unless>
+                <joint name="joint1">
+                    <command_interface name="position"/>
+                    <state_interface name="position">
+                        <param name="initial_value">${initial_positions['joint1']}</param>
+                    </state_interface>
+                </joint>
+                <joint name="joint2">
+                    <command_interface name="position"/>
+                    <state_interface name="position">
+                        <param name="initial_value">${initial_positions['joint2']}</param>
+                    </state_interface>
+                </joint>
+                <joint name="joint3">
+                    <command_interface name="position"/>
+                    <state_interface name="position">
+                        <param name="initial_value">${initial_positions['joint3']}</param>
+                    </state_interface>
+                </joint>
+                <joint name="joint4">
+                    <command_interface name="position"/>
+                    <state_interface name="position">
+                        <param name="initial_value">${initial_positions['joint4']}</param>
+                    </state_interface>
+                </joint>
+                <joint name="joint5">
+                    <command_interface name="position"/>
+                    <state_interface name="position">
+                        <param name="initial_value">${initial_positions['joint5']}</param>
+                    </state_interface>
+                </joint>
+                <joint name="joint6">
+                    <command_interface name="position"/>
+                    <state_interface name="position">
+                        <param name="initial_value">${initial_positions['joint6']}</param>
+                    </state_interface>
+                </joint>
+                <joint name="gripper_left_finger_joint">
+                    <command_interface name="position"/>
+                    <state_interface name="position">
+                        <param name="initial_value">${initial_positions['gripper_left_finger_joint']}</param>
+                    </state_interface>
+                </joint>
+            </ros2_control>
+        </xacro:macro>
+    </robot>
