Commit message: update code

File: src/my_robot_description/urdf/amr.xacro (robot description, xacro)
@@ -1,5 +1,5 @@
 <?xml version="1.0"?>
 <robot xmlns:xacro="http://www.ros.org/wiki/xacro">
-    <link name="base_link">
+    <link name="base_arm_link">
         <visual>
             <geometry>
@@ -16,35 +16,5 @@
         </collision>
     </link>
-    <link name="shoulder_link">
-        <visual>
-            <geometry>
-                <cylinder radius="0.1" length="0.5"/>
-            </geometry>
-            <origin xyz="0.0 0.0 0.25" rpy="0.0 0.0 0.0"/>
-            <material name="blue"/>
-        </visual>
-        <collision>
-            <geometry>
-                <box size="0.2 0.2 0.5"/>
-            </geometry>
-            <origin xyz="0.0 0.0 0.25" rpy="0.0 0.0 0.0"/>
-        </collision>
-    </link>
     <link name="amr_link">
-        <visual>
-            <geometry>
-                <cylinder radius="0.05" length="0.6"/>
-            </geometry>
-            <origin xyz="0.0 0.0 0.3" rpy="0.0 0.0 0.0"/>
-            <material name="grey"/>
-        </visual>
-        <collision>
-            <geometry>
-                <box size="0.1 0.1 0.6"/>
-            </geometry>
-            <origin xyz="0.0 0.0 0.3" rpy="0.0 0.0 0.0"/>
-        </collision>
-    </link>
-    <link name="elbow_link">
         <visual>
             <geometry>
@@ -52,5 +22,5 @@
             </geometry>
             <origin xyz="0.0 0.0 0.05" rpy="0.0 0.0 0.0"/>
-            <material name="blue"/>
+            <material name="dark_green"/>
         </visual>
         <collision>
@@ -64,32 +34,17 @@
         <visual>
             <geometry>
-                <cylinder radius="0.05" length="0.5"/>
+                <cylinder radius="0.05" length="0.2"/>
             </geometry>
-            <origin xyz="0.0 0.0 0.25" rpy="0.0 0.0 0.0"/>
-            <material name="grey"/>
+            <origin xyz="0.0 0.0 0.1" rpy="0.0 0.0 0.0"/>
+            <material name="light_green"/>
         </visual>
         <collision>
             <geometry>
-                <box size="0.1 0.1 0.5"/>
+                <box size="0.1 0.1 0.2"/>
             </geometry>
-            <origin xyz="0.0 0.0 0.25" rpy="0.0 0.0 0.0"/>
+            <origin xyz="0.0 0.0 0.1" rpy="0.0 0.0 0.0"/>
         </collision>
     </link>
-    <link name="wrist_link">
-        <visual>
-            <geometry>
-                <box size="0.1 0.1 0.05"/>
-            </geometry>
-            <origin xyz="0.0 0.0 0.025" rpy="0.0 0.0 0.0"/>
-            <material name="blue"/>
-        </visual>
-        <collision>
-            <geometry>
-                <box size="0.1 0.1 0.05"/>
-            </geometry>
-            <origin xyz="0.0 0.0 0.025" rpy="0.0 0.0 0.0"/>
-        </collision>
-    </link>
-     <link name="hand_link">
+    <link name="hand_link">
         <visual>
             <geometry>
@@ -97,5 +52,5 @@
             </geometry>
             <origin xyz="0.0 0.0 0.01" rpy="0.0 0.0 0.0"/>
-            <material name="grey"/>
+            <material name="blue"/>
         </visual>
         <collision>
@@ -110,43 +65,22 @@
     <joint name="joint1" type="revolute">
         <origin xyz="0.0 0.0 0.1" rpy="0.0 0.0 0.0"/>
-        <parent link="base_link"/>
-        <child link="shoulder_link"/>
+        <parent link="base_arm_link"/>
+        <child link="amr_link"/>
         <axis xyz="0.0 0.0 1.0"/>
-        <limit lower="-3.14" upper="3.14" effort="1000.0" velocity="1.0"/>
+        <limit lower="-1.57" upper="1.57" effort="1000.0" velocity="1.0"/>
     </joint>
     <joint name="joint2" type="revolute">
-        <origin xyz="0.0 0.0 0.5" rpy="0.0 0.0 0.0"/>
-        <parent link="shoulder_link"/>
-        <child link="amr_link"/>
+        <origin xyz="0.0 0.0 0.1" rpy="0.0 0.0 0.0"/>
+        <parent link="amr_link"/>
+        <child link="forearm_link"/>
         <axis xyz="0.0 1.0 0.0"/>
-        <limit lower="0" upper="2.5" effort="1000.0" velocity="1.0"/>
+        <limit lower="-1.57" upper="1.57" effort="1000.0" velocity="1.0"/>
     </joint>
     <joint name="joint3" type="revolute">
-        <origin xyz="0.0 0.0 0.6" rpy="0.0 0.0 0.0"/>
-        <parent link="amr_link"/>
-        <child link="elbow_link"/>
-        <axis xyz="0.0 1.0 0.0"/>
-        <limit lower="0" upper="2.5" effort="1000.0" velocity="1.0"/>
-    </joint>
-    <joint name="joint4" type="revolute">
-        <origin xyz="0.0 0.0 0.1" rpy="0.0 0.0 0.0"/>
-        <parent link="elbow_link"/>
-        <child link="forearm_link"/>
+        <origin xyz="0.0 0.0 0.2" rpy="0.0 0.0 0.0"/>
+        <parent link="forearm_link"/>
+        <child link="hand_link"/>
         <axis xyz="0.0 0.0 1.0"/>
-        <limit lower="-3.14" upper="3.14" effort="1000.0" velocity="1.0"/>
-    </joint>
-    <joint name="joint5" type="revolute">
-        <origin xyz="0.0 0.0 0.5" rpy="0.0 0.0 0.0"/>
-        <parent link="forearm_link"/>
-        <child link="wrist_link"/>
-         <axis xyz="0.0 1.0 0.0"/>
         <limit lower="-1.57" upper="1.57" effort="1000.0" velocity="1.0"/>
-    </joint>
-    <joint name="joint6" type="continuous">
-        <origin xyz="0.0 0.0 0.05" rpy="0.0 0.0 0.0"/>
-        <parent link="wrist_link"/>
-        <child link="hand_link"/>
-         <axis xyz="0.0 0.0 1.0"/>
-        <limit  effort="1000.0" velocity="1.0"/>
     </joint>
     <joint name="hand_tool_joint" type="fixed">

File: src/my_robot_description/urdf/my_robot.ros2_control.xacro (robot description, xacro)
@@ -4,14 +4,6 @@
     <ros2_control name="Amr" type="system">
         <!-- <hardware>
-          <xacro:if value="$(arg use_mock_component)">
             <plugin>mock_components/GenericSystem</plugin>
-          </xacro:if>
-          <xacro:unless value="$(arg use_mock_component)">
-            <plugin>arm_hardware/ArmHardwareInterface</plugin>
-            <param name="joint1_motor_id">10</param>
-            <param name="joint2_motor_id">20</param>
-            <param name="dynamixel_port">/dev/ttyACM0</param>
-          </xacro:unless>
-      </hardware> -->
+        </hardware> -->
         <hardware>
             <xacro:if value="$(arg use_mock_component)">
@@ -25,7 +17,4 @@
                 <param name="joint2_channel">2</param>
                 <param name="joint3_channel">3</param>
-                <param name="joint4_channel">4</param>
-                <param name="joint5_channel">5</param>
-                <param name="joint6_channel">6</param>
                 <param name="gripper_channel">0</param>
             </xacro:unless>
@@ -49,22 +38,4 @@
             </state_interface>
         </joint>
-        <joint name="joint4">
-            <command_interface name="position"/>
-            <state_interface name="position">
-                <param name="initial_value">0.0</param>
-            </state_interface>
-        </joint>
-        <joint name="joint5">
-            <command_interface name="position"/>
-            <state_interface name="position">
-                <param name="initial_value">0.0</param>
-            </state_interface>
-        </joint>
-        <joint name="joint6">
-            <command_interface name="position"/>
-            <state_interface name="position">
-                <param name="initial_value">0.0</param>
-            </state_interface>
-        </joint>
         <joint name="gripper_left_finger_joint">
             <command_interface name="position"/>

File: src/my_robot_moveit_config/config/my_robot.ros2_control.xacro (robot description, xacro)
@@ -8,47 +8,29 @@
                 <plugin>mock_components/GenericSystem</plugin>
             </hardware>
-                <joint name="joint1">
-                    <command_interface name="position"/>
-                    <state_interface name="position">
-                        <param name="initial_value">${initial_positions['joint1']}</param>
-                    </state_interface>
-                </joint>
-                <joint name="joint2">
-                    <command_interface name="position"/>
-                    <state_interface name="position">
-                        <param name="initial_value">${initial_positions['joint2']}</param>
-                    </state_interface>
-                </joint>
-                <joint name="joint3">
-                    <command_interface name="position"/>
-                    <state_interface name="position">
-                        <param name="initial_value">${initial_positions['joint3']}</param>
-                    </state_interface>
-                </joint>
-                <joint name="joint4">
-                    <command_interface name="position"/>
-                    <state_interface name="position">
-                        <param name="initial_value">${initial_positions['joint4']}</param>
-                    </state_interface>
-                </joint>
-                <joint name="joint5">
-                    <command_interface name="position"/>
-                    <state_interface name="position">
-                        <param name="initial_value">${initial_positions['joint5']}</param>
-                    </state_interface>
-                </joint>
-                <joint name="joint6">
-                    <command_interface name="position"/>
-                    <state_interface name="position">
-                        <param name="initial_value">${initial_positions['joint6']}</param>
-                    </state_interface>
-                </joint>
-                <joint name="gripper_left_finger_joint">
-                    <command_interface name="position"/>
-                    <state_interface name="position">
-                        <param name="initial_value">${initial_positions['gripper_left_finger_joint']}</param>
-                    </state_interface>
-                </joint>
-            </ros2_control>
-        </xacro:macro>
-    </robot>
+            <joint name="joint1">
+                <command_interface name="position"/>
+                <state_interface name="position">
+                  <param name="initial_value">${initial_positions['joint1']}</param>
+                </state_interface>
+            </joint>
+            <joint name="joint2">
+                <command_interface name="position"/>
+                <state_interface name="position">
+                  <param name="initial_value">${initial_positions['joint2']}</param>
+                </state_interface>
+            </joint>
+            <joint name="joint3">
+                <command_interface name="position"/>
+                <state_interface name="position">
+                  <param name="initial_value">${initial_positions['joint3']}</param>
+                </state_interface>
+            </joint>
+            <joint name="gripper_left_finger_joint">
+                <command_interface name="position"/>
+                <state_interface name="position">
+                  <param name="initial_value">${initial_positions['gripper_left_finger_joint']}</param>
+                </state_interface>
+            </joint>
+        </ros2_control>
+    </xacro:macro>
+</robot>

Commit message: add joint 4

File: src/my_robot_description/urdf/amr.xacro (robot description, xacro)
@@ -1,4 +1,16 @@
 <?xml version="1.0"?>
 <robot xmlns:xacro="http://www.ros.org/wiki/xacro">
+    <!-- <material name="grey">
+        <color rgba="0.5 0.5 0.5 1.0"/>
+    </material>
+    <material name="blue">
+        <color rgba="0.0 0.0 0.5 1.0"/>
+    </material>
+    <material name="dark_green">
+        <color rgba="0.0 0.4 0 1"/>
+    </material>
+    <material name="light_green">
+        <color rgba="0.0 1.0 0 1"/>
+    </material> -->
     <link name="base_arm_link">
         <visual>
@@ -34,14 +46,29 @@
         <visual>
             <geometry>
-                <cylinder radius="0.05" length="0.2"/>
+                <cylinder radius="0.05" length="0.1"/>
             </geometry>
-            <origin xyz="0.0 0.0 0.1" rpy="0.0 0.0 0.0"/>
+            <origin xyz="0.0 0.0 0.05" rpy="0.0 0.0 0.0"/>
             <material name="light_green"/>
         </visual>
         <collision>
             <geometry>
-                <box size="0.1 0.1 0.2"/>
+                <box size="0.1 0.1 0.1"/>
             </geometry>
-            <origin xyz="0.0 0.0 0.1" rpy="0.0 0.0 0.0"/>
+            <origin xyz="0.0 0.0 0.05" rpy="0.0 0.0 0.0"/>
+        </collision>
+    </link>
+    <link name="forearm_link2">
+        <visual>
+            <geometry>
+                <cylinder radius="0.05" length="0.1"/>
+            </geometry>
+            <origin xyz="0.0 0.0 0.05" rpy="0.0 0.0 0.0"/>
+            <material name="grey"/>
+        </visual>
+        <collision>
+            <geometry>
+                <box size="0.1 0.1 0.1"/>
+            </geometry>
+            <origin xyz="0.0 0.0 0.05" rpy="0.0 0.0 0.0"/>
         </collision>
     </link>
@@ -78,6 +105,13 @@
     </joint>
     <joint name="joint3" type="revolute">
-        <origin xyz="0.0 0.0 0.2" rpy="0.0 0.0 0.0"/>
+        <origin xyz="0.0 0.0 0.1" rpy="0.0 0.0 0.0"/>
         <parent link="forearm_link"/>
+        <child link="forearm_link2"/>
+        <axis xyz="0.0 1.0 0.0"/>
+        <limit lower="-1.57" upper="1.57" effort="1000.0" velocity="1.0"/>
+    </joint>
+    <joint name="joint4" type="revolute">
+        <origin xyz="0.0 0.0 0.1" rpy="0.0 0.0 0.0"/>
+        <parent link="forearm_link2"/>
         <child link="hand_link"/>
         <axis xyz="0.0 0.0 1.0"/>

File: src/my_robot_description/urdf/my_robot.ros2_control.xacro (robot description, xacro)
@@ -17,4 +17,5 @@
                 <param name="joint2_channel">2</param>
                 <param name="joint3_channel">3</param>
+                <param name="joint4_channel">4</param>
                 <param name="gripper_channel">0</param>
             </xacro:unless>
@@ -38,4 +39,10 @@
             </state_interface>
         </joint>
+        <joint name="joint4">
+            <command_interface name="position"/>
+            <state_interface name="position">
+                <param name="initial_value">0.0</param>
+            </state_interface>
+        </joint>
         <joint name="gripper_left_finger_joint">
             <command_interface name="position"/>

File: src/my_robot_moveit_config/config/my_robot.ros2_control.xacro (robot description, xacro)
@@ -2,5 +2,5 @@
 <robot xmlns:xacro="http://www.ros.org/wiki/xacro">
     <xacro:macro name="my_robot_ros2_control" params="name initial_positions_file">
-        <xacro:property name="initial_positions" value="${xacro.load_yaml(initial_positions_file)['initial_positions']}"/>
+        <xacro:property name="initial_positions" value="${load_yaml(initial_positions_file)['initial_positions']}"/>
         <ros2_control name="${name}" type="system">
             <hardware>
@@ -26,4 +26,10 @@
                 </state_interface>
             </joint>
+            <joint name="joint4">
+                <command_interface name="position"/>
+                <state_interface name="position">
+                  <param name="initial_value">${initial_positions['joint4']}</param>
+                </state_interface>
+            </joint>
             <joint name="gripper_left_finger_joint">
                 <command_interface name="position"/>

Commit message: update code

File: src/my_robot_description/urdf/amr.xacro (robot description, xacro)
@@ -61,7 +61,7 @@
         <visual>
             <geometry>
-                <cylinder radius="0.05" length="0.1"/>
+                <cylinder radius="0.05" length="0.2"/>
             </geometry>
-            <origin xyz="0.0 0.0 0.05" rpy="0.0 0.0 0.0"/>
+            <origin xyz="0.0 0.0 0.1" rpy="0.0 0.0 0.0"/>
             <material name="grey"/>
         </visual>
@@ -70,5 +70,5 @@
                 <box size="0.1 0.1 0.1"/>
             </geometry>
-            <origin xyz="0.0 0.0 0.05" rpy="0.0 0.0 0.0"/>
+            <origin xyz="0.0 0.0 0.1" rpy="0.0 0.0 0.0"/>
         </collision>
     </link>
@@ -112,5 +112,5 @@
     </joint>
     <joint name="joint4" type="revolute">
-        <origin xyz="0.0 0.0 0.1" rpy="0.0 0.0 0.0"/>
+        <origin xyz="0.0 0.0 0.2" rpy="0.0 0.0 0.0"/>
         <parent link="forearm_link2"/>
         <child link="hand_link"/>

Commit message: add joint 5

File: src/my_robot_description/urdf/amr.xacro (robot description, xacro)
@@ -61,7 +61,7 @@
         <visual>
             <geometry>
-                <cylinder radius="0.05" length="0.2"/>
+                <cylinder radius="0.05" length="0.1"/>
             </geometry>
-            <origin xyz="0.0 0.0 0.1" rpy="0.0 0.0 0.0"/>
+            <origin xyz="0.0 0.0 0.05" rpy="0.0 0.0 0.0"/>
             <material name="grey"/>
         </visual>
@@ -70,5 +70,20 @@
                 <box size="0.1 0.1 0.1"/>
             </geometry>
-            <origin xyz="0.0 0.0 0.1" rpy="0.0 0.0 0.0"/>
+            <origin xyz="0.0 0.0 0.05" rpy="0.0 0.0 0.0"/>
+        </collision>
+    </link>
+     <link name="forearm_link3">
+        <visual>
+            <geometry>
+                <cylinder radius="0.05" length="0.1"/>
+            </geometry>
+            <origin xyz="0.0 0.0 0.05" rpy="0.0 0.0 0.0"/>
+            <material name="grey"/>
+        </visual>
+        <collision>
+            <geometry>
+                <box size="0.1 0.1 0.1"/>
+            </geometry>
+            <origin xyz="0.0 0.0 0.05" rpy="0.0 0.0 0.0"/>
         </collision>
     </link>
@@ -112,6 +127,13 @@
     </joint>
     <joint name="joint4" type="revolute">
-        <origin xyz="0.0 0.0 0.2" rpy="0.0 0.0 0.0"/>
+        <origin xyz="0.0 0.0 0.1" rpy="0.0 0.0 0.0"/>
         <parent link="forearm_link2"/>
+        <child link="forearm_link3"/>
+        <axis xyz="0.0 1.0 0.0"/>
+        <limit lower="-1.57" upper="1.57" effort="1000.0" velocity="1.0"/>
+    </joint>
+     <joint name="joint5" type="revolute">
+        <origin xyz="0.0 0.0 0.1" rpy="0.0 0.0 0.0"/>
+        <parent link="forearm_link3"/>
         <child link="hand_link"/>
         <axis xyz="0.0 0.0 1.0"/>

File: src/my_robot_description/urdf/my_robot.ros2_control.xacro (robot description, xacro)
@@ -1,5 +1,5 @@
 <?xml version="1.0"?>
 <robot xmlns:xacro="http://www.ros.org/wiki/xacro">
-    <xacro:arg name="use_mock_component" default="true"/>
+    <xacro:arg name="use_sim" default="true"/>
     <ros2_control name="Amr" type="system">
         <!-- <hardware>
@@ -7,8 +7,8 @@
         </hardware> -->
         <hardware>
-            <xacro:if value="$(arg use_mock_component)">
+            <xacro:if value="$(arg use_sim)">
                 <plugin>mock_components/GenericSystem</plugin>
             </xacro:if>
-            <xacro:unless value="$(arg use_mock_component)">
+            <xacro:unless value="$(arg use_sim)">
                 <plugin>arm_hardware/ArmHardwareInterface</plugin>
                 <param name="serial_port">/dev/serial/by-id/usb-Espressif_USB_JTAG_serial_debug_unit_3C:DC:75:62:AD:B8-if00</param>
@@ -18,4 +18,5 @@
                 <param name="joint3_channel">3</param>
                 <param name="joint4_channel">4</param>
+                <param name="joint4_channel">5</param>
                 <param name="gripper_channel">0</param>
             </xacro:unless>
@@ -45,4 +46,10 @@
             </state_interface>
         </joint>
+        <joint name="joint5">
+            <command_interface name="position"/>
+            <state_interface name="position">
+                <param name="initial_value">0.0</param>
+            </state_interface>
+        </joint>
         <joint name="gripper_left_finger_joint">
             <command_interface name="position"/>

File: src/my_robot_moveit_config/config/my_robot.ros2_control.xacro (robot description, xacro)
@@ -2,5 +2,5 @@
 <robot xmlns:xacro="http://www.ros.org/wiki/xacro">
     <xacro:macro name="my_robot_ros2_control" params="name initial_positions_file">
-        <xacro:property name="initial_positions" value="${load_yaml(initial_positions_file)['initial_positions']}"/>
+        <xacro:property name="initial_positions" value="${xacro.load_yaml(initial_positions_file)['initial_positions']}"/>
         <ros2_control name="${name}" type="system">
             <hardware>
@@ -32,4 +32,10 @@
                 </state_interface>
             </joint>
+            <joint name="joint5">
+                <command_interface name="position"/>
+                <state_interface name="position">
+                  <param name="initial_value">${initial_positions['joint5']}</param>
+                </state_interface>
+            </joint>
             <joint name="gripper_left_finger_joint">
                 <command_interface name="position"/>
